Commit message: Organizing common folder.

File: common/urdfs/Ramp.urdf (robot description, URDF)
Before this commit: robot simple_ball, 1 links, 0 joints
Links:
- removed link ball
- added link ramp, mass 1.0; collision mesh filename=../meshes/Ramp.obj scale=1 1 1; visual mesh filename=../meshes/Ramp.obj scale=1 1 1

File: common/urdfs/sphere.urdf (robot description, URDF)
Before this commit: robot simple_ramp, 1 links, 0 joints
Links:
- removed link ramp
- added link ball, mass 1.0; collision mesh filename=../meshes/sphere.obj scale=1 1 1; visual mesh filename=../meshes/sphere.obj scale=1 1 1
